File: eagle/schem.brd (EAGLE design)
At the start: 100 x 40 mm, 7 parts, among them U1 WIFI-LORA-32-V2

Commit message: fix eagle files
Parts:
- removed J1, J2, J3, J4: (no value), ME433-2021:1X09
Connections:
- net GND: no longer J3.5, J4.6
Changed lines of the file:
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@@
 <attribute name="VALUE" x="66.04" y="5.588" size="0.6096" layer="27" font="vector" ratio="20"/>
-</element>
-<element name="J1" library="ME433-2021" package="1X09" value="" x="6.35" y="35.56" smashed="yes">
-<attribute name="NAME" x="5.08" y="36.957" size="0.6096" layer="25" font="vector" ratio="20"/>
-<attribute name="VALUE" x="5.08" y="33.528" size="0.6096" layer="27" font="vector" ratio="20"/>
-</element>
-<element name="J2" library="ME433-2021" package="1X09" value="" x="29.21" y="35.56" smashed="yes">
-<attribute name="NAME" x="27.94" y="36.957" size="0.6096" layer="25" font="vector" ratio="20"/>
-<attribute name="VALUE" x="27.94" y="33.528" size="0.6096" layer="27" font="vector" ratio="20"/>
-</element>
-<element name="J3" library="ME433-2021" package="1X09" value="" x="6.35" y="3.81" smashed="yes">
-<attribute name="NAME" x="5.08" y="5.207" size="0.6096" layer="25" font="vector" ratio="20"/>
-<attribute name="VALUE" x="5.08" y="1.778" size="0.6096" layer="27" font="vector" ratio="20"/>
-</element>
-<element name="J4" library="ME433-2021" package="1X09" value="" x="29.21" y="3.81" smashed="yes">
-<attribute name="NAME" x="27.94" y="5.207" size="0.6096" layer="25" font="vector" ratio="20"/>
-<attribute name="VALUE" x="27.94" y="1.778" size="0.6096" layer="27" font="vector" ratio="20"/>
 </element>
 <element name="U1" library="telemetry_module" package="2.54MM_2X18" value="WIFI-LORA-32-V2" x="26.67" y="19.05" smashed="yes">
@@
 <vertex x="0.127" y="-0.127"/>
 </polygon>
-<contactref element="J3" pad="5"/>
 <contactref element="U1" pad="P$1"/>
-<contactref element="J4" pad="6"/>
 <contactref element="U1" pad="P$36"/>
 </signal>
